File: rc2014-ym2149.sch (KiCad schematic (older format))
At the start: 28 parts, among them J1 AUDIO OUT, J2 IO Out, P1 RC2014 BUS, U1 74HCT138, U2 74HCT138, U3 74HCT00, U4 74HCT74, U5 AY-3-8190/YM2149F

Commit message: Update pulldown values to 3k
Parts:
- R1, R2, R3: value 470R -> 3K
Changed lines of the file:
@@
 P 7600 1350
 F 0 "R2" H 7630 1370 50  0000 L CNN
-F 1 "470R" H 7630 1310 50  0000 L CNN
+F 1 "3K" H 7630 1310 50  0000 L CNN
 F 2 "rc2014:R_Axial_DIN0207_L6.3mm_D2.5mm_P10.16mm_Horizontal" H 7600 1350 50  0001 C CNN
 F 3 "" H 7600 1350 50  0000 C CNN
@@
 P 7300 1350
 F 0 "R1" H 7330 1370 50  0000 L CNN
-F 1 "470R" H 7330 1310 50  0000 L CNN
+F 1 "3K" H 7330 1310 50  0000 L CNN
 F 2 "rc2014:R_Axial_DIN0207_L6.3mm_D2.5mm_P10.16mm_Horizontal" H 7300 1350 50  0001 C CNN
 F 3 "" H 7300 1350 50  0000 C CNN
@@
 P 7900 1350
 F 0 "R3" H 7930 1370 50  0000 L CNN
-F 1 "470R" H 7930 1310 50  0000 L CNN
+F 1 "3K" H 7930 1310 50  0000 L CNN
 F 2 "rc2014:R_Axial_DIN0207_L6.3mm_D2.5mm_P10.16mm_Horizontal" H 7900 1350 50  0001 C CNN
 F 3 "" H 7900 1350 50  0000 C CNN

Commit message: Rev 5
Parts:
- C1, C2, C3, C4, C5: footprint Capacitors_THT:C_Disc_D3.8mm_W2.6mm_P2.50mm -> rc2014:C_Disc_D3.8mm_W2.6mm_P2.50mm
- C6, C7: footprint Capacitors_THT:CP_Radial_D5.0mm_P2.50mm -> Capacitors_THT:CP_Radial_D6.3mm_P2.50mm
- J2: footprint Pin_Headers:Pin_Header_Straight_2x09_Pitch2.54mm -> rc2014:Pin_Header_Straight_2x09_Pitch2.54mm
- JP1, JP2, JP5: footprint Pin_Headers:Pin_Header_Straight_1x03_Pitch2.54mm -> rc2014:Pin_Header_Straight_1x03_Pitch2.54mm
- JP3: footprint Pin_Headers:Pin_Header_Straight_2x03_Pitch2.54mm -> rc2014:Pin_Header_Straight_2x03_Pitch2.54mm
- JP4: footprint Pin_Headers:Pin_Header_Straight_2x08_Pitch2.54mm -> rc2014:Pin_Header_Straight_2x08_Pitch2.54mm
- JP6: footprint Pin_Headers:Pin_Header_Straight_1x02_Pitch2.54mm -> rc2014:Pin_Header_Straight_1x02_Pitch2.54mm
- U1, U2: footprint Housings_DIP:DIP-16_W7.62mm_Socket -> rc2014:DIP-16_W7.62mm_Socket
- U3, U4: footprint Housings_DIP:DIP-14_W7.62mm_Socket -> rc2014:DIP-14_W7.62mm_Socket
- U5: footprint Housings_DIP:DIP-40_W15.24mm_Socket -> rc2014:DIP-40_W15.24mm_Socket
Changed lines of the file:
@@
 F 0 "U5" H 6600 4150 50  0000 C CNN
 F 1 "AY-3-8190/YM2149F" V 6600 3100 50  0000 C CNN
-F 2 "Housings_DIP:DIP-40_W15.24mm_Socket" H 6600 3100 50  0001 C CNN
+F 2 "rc2014:DIP-40_W15.24mm_Socket" H 6600 3100 50  0001 C CNN
 F 3 "" H 6600 3100 50  0000 C CNN
 	1    6600 3100
@@
 F 0 "U2" H 3550 3700 50  0000 C CNN
 F 1 "74HCT138" H 3600 2651 50  0000 C CNN
-F 2 "Housings_DIP:DIP-16_W7.62mm_Socket" H 3450 3200 50  0001 C CNN
+F 2 "rc2014:DIP-16_W7.62mm_Socket" H 3450 3200 50  0001 C CNN
 F 3 "" H 3450 3200 50  0000 C CNN
 F 4 "CD74HCT138E" H 3450 3200 60  0001 C CNN "MPN"
@@
 F 0 "U4" H 5850 5600 50  0000 C CNN
 F 1 "74HCT74" H 6000 5005 50  0000 C CNN
-F 2 "Housings_DIP:DIP-14_W7.62mm_Socket" H 5700 5300 50  0001 C CNN
+F 2 "rc2014:DIP-14_W7.62mm_Socket" H 5700 5300 50  0001 C CNN
 F 3 "" H 5700 5300 50  0000 C CNN
 F 4 "SN74HCT74N" H 5700 5300 60  0001 C CNN "MPN"
@@
 F 0 "C5" H 7225 2100 50  0000 L CNN
 F 1 "0.1uF" H 7225 1900 50  0000 L CNN
-F 2 "Capacitors_THT:C_Disc_D3.8mm_W2.6mm_P2.50mm" H 7238 1850 50  0001 C CNN
+F 2 "rc2014:C_Disc_D3.8mm_W2.6mm_P2.50mm" H 7238 1850 50  0001 C CNN
 F 3 "" H 7200 2000 50  0000 C CNN
 	1    7200 2000
@@
 F 0 "U3" H 4950 3150 50  0000 C CNN
 F 1 "74HCT00" H 4950 3000 50  0000 C CNN
-F 2 "Housings_DIP:DIP-14_W7.62mm_Socket" H 4950 3100 50  0001 C CNN
+F 2 "rc2014:DIP-14_W7.62mm_Socket" H 4950 3100 50  0001 C CNN
 F 3 "" H 4950 3100 50  0000 C CNN
 	1    4950 3100
@@
 F 0 "U3" H 4950 3700 50  0000 C CNN
 F 1 "74HCT00" H 4950 3550 50  0000 C CNN
-F 2 "Housings_DIP:DIP-14_W7.62mm_Socket" H 4950 3650 50  0001 C CNN
+F 2 "rc2014:DIP-14_W7.62mm_Socket" H 4950 3650 50  0001 C CNN
 F 3 "" H 4950 3650 50  0000 C CNN
 	2    4950 3650
@@
 F 0 "JP6" H 8650 3700 50  0000 C CNN
 F 1 "YM 1/2 CLK" H 8650 3470 50  0000 C CNN
-F 2 "Pin_Headers:Pin_Header_Straight_1x02_Pitch2.54mm" H 8650 3550 50  0001 C CNN
+F 2 "rc2014:Pin_Header_Straight_1x02_Pitch2.54mm" H 8650 3550 50  0001 C CNN
 F 3 "" H 8650 3550 50  0000 C CNN
 	1    8650 3550
@@
 F 0 "U4" H 5850 7150 50  0000 C CNN
 F 1 "74HCT74" H 6000 6555 50  0000 C CNN
-F 2 "Housings_DIP:DIP-14_W7.62mm_Socket" H 5700 6850 50  0001 C CNN
+F 2 "rc2014:DIP-14_W7.62mm_Socket" H 5700 6850 50  0001 C CNN
 F 3 "" H 5700 6850 50  0000 C CNN
 	2    5700 6850
@@
 F 0 "J2" H 10450 3100 50  0000 C CNN
 F 1 "IO Out" V 10450 2600 50  0000 C CNN
-F 2 "Pin_Headers:Pin_Header_Straight_2x09_Pitch2.54mm" H 10450 1400 50  0001 C CNN
+F 2 "rc2014:Pin_Header_Straight_2x09_Pitch2.54mm" H 10450 1400 50  0001 C CNN
 F 3 "" H 10450 1400 50  0000 C CNN
 	1    10450 2600
@@
 F 0 "C6" H 9025 900 50  0000 L CNN
 F 1 "470uF" H 9025 700 50  0000 L CNN
-F 2 "Capacitors_THT:CP_Radial_D5.0mm_P2.50mm" H 9038 650 50  0001 C CNN
+F 2 "Capacitors_THT:CP_Radial_D6.3mm_P2.50mm" H 9038 650 50  0001 C CNN
 F 3 "" H 9000 800 50  0000 C CNN
 	1    9000 800
@@
 F 0 "C7" H 9025 1100 50  0000 L CNN
 F 1 "470uF" H 9025 900 50  0000 L CNN
-F 2 "Capacitors_THT:CP_Radial_D5.0mm_P2.50mm" H 9038 850 50  0001 C CNN
+F 2 "Capacitors_THT:CP_Radial_D6.3mm_P2.50mm" H 9038 850 50  0001 C CNN
 F 3 "" H 9000 1000 50  0000 C CNN
 	1    9000 1000
@@
 F 0 "C1" H 2575 6500 50  0000 L CNN
 F 1 "C" H 2575 6300 50  0000 L CNN
-F 2 "Capacitors_THT:C_Disc_D3.8mm_W2.6mm_P2.50mm" H 2588 6250 50  0001 C CNN
+F 2 "rc2014:C_Disc_D3.8mm_W2.6mm_P2.50mm" H 2588 6250 50  0001 C CNN
 F 3 "" H 2550 6400 50  0001 C CNN
 	1    2550 6400
@@
 F 0 "C2" H 2925 6500 50  0000 L CNN
 F 1 "C" H 2925 6300 50  0000 L CNN
-F 2 "Capacitors_THT:C_Disc_D3.8mm_W2.6mm_P2.50mm" H 2938 6250 50  0001 C CNN
+F 2 "rc2014:C_Disc_D3.8mm_W2.6mm_P2.50mm" H 2938 6250 50  0001 C CNN
 F 3 "" H 2900 6400 50  0001 C CNN
 	1    2900 6400
@@
 F 0 "C3" H 3275 6500 50  0000 L CNN
 F 1 "C" H 3275 6300 50  0000 L CNN
-F 2 "Capacitors_THT:C_Disc_D3.8mm_W2.6mm_P2.50mm" H 3288 6250 50  0001 C CNN
+F 2 "rc2014:C_Disc_D3.8mm_W2.6mm_P2.50mm" H 3288 6250 50  0001 C CNN
 F 3 "" H 3250 6400 50  0001 C CNN
 	1    3250 6400
@@
 F 0 "JP5" H 7500 5250 50  0000 L CNN
 F 1 "CLOCK DIVIDE 1/2 or 1/4" H 7450 5450 50  0000 C BNN
-F 2 "Pin_Headers:Pin_Header_Straight_1x03_Pitch2.54mm" H 7450 5350 50  0001 C CNN
+F 2 "rc2014:Pin_Header_Straight_1x03_Pitch2.54mm" H 7450 5350 50  0001 C CNN
 F 3 "" H 7450 5350 50  0001 C CNN
 	1    7450 5350
@@
 F 0 "JP3" H 2300 2900 50  0000 C CNN
 F 1 "CONN_02X03" H 2300 2500 50  0000 C CNN
-F 2 "Pin_Headers:Pin_Header_Straight_2x03_Pitch2.54mm" H 2300 1500 50  0001 C CNN
+F 2 "rc2014:Pin_Header_Straight_2x03_Pitch2.54mm" H 2300 1500 50  0001 C CNN
 F 3 "" H 2300 1500 50  0001 C CNN
 	1    2300 2700
@@
 F 0 "JP4" H 3550 1600 50  0000 C CNN
 F 1 "BASE ADDRESS" V 3550 1150 50  0000 C CNN
-F 2 "Pin_Headers:Pin_Header_Straight_2x08_Pitch2.54mm" H 3550 -50 50  0001 C CNN
+F 2 "rc2014:Pin_Header_Straight_2x08_Pitch2.54mm" H 3550 -50 50  0001 C CNN
 F 3 "" H 3550 -50 50  0001 C CNN
 	1    3550 1150
@@
 F 0 "U1" H 2650 1650 50  0000 C CNN
 F 1 "74HCT138" H 2700 601 50  0000 C CNN
-F 2 "Housings_DIP:DIP-16_W7.62mm_Socket" H 2550 1150 50  0001 C CNN
+F 2 "rc2014:DIP-16_W7.62mm_Socket" H 2550 1150 50  0001 C CNN
 F 3 "" H 2550 1150 50  0000 C CNN
 F 4 "CD74HCT138E" H 2550 1150 60  0001 C CNN "MPN"
@@
 F 0 "JP1" H 1100 1250 50  0000 C CNN
 F 1 "USE A4 FOR ENABLE" H 1150 800 50  0000 C CNN
-F 2 "Pin_Headers:Pin_Header_Straight_1x03_Pitch2.54mm" H 1100 -100 50  0001 C CNN
+F 2 "rc2014:Pin_Header_Straight_1x03_Pitch2.54mm" H 1100 -100 50  0001 C CNN
 F 3 "" H 1100 -100 50  0001 C CNN
 F 4 "CONN 1x03" H 1100 1100 60  0001 C CNN "MPN"
@@
 F 0 "JP2" H 2250 3350 50  0000 C CNN
 F 1 "ENABLE SELECTOR" H 2250 2850 50  0000 C CNN
-F 2 "Pin_Headers:Pin_Header_Straight_1x03_Pitch2.54mm" H 2250 2000 50  0001 C CNN
+F 2 "rc2014:Pin_Header_Straight_1x03_Pitch2.54mm" H 2250 2000 50  0001 C CNN
 F 3 "" H 2250 2000 50  0001 C CNN
 	1    2250 3200
@@
 F 0 "U3" H 5050 1200 50  0000 C CNN
 F 1 "74HCT00" H 5050 1050 50  0000 C CNN
-F 2 "Housings_DIP:DIP-14_W7.62mm_Socket" H 5050 1150 50  0001 C CNN
+F 2 "rc2014:DIP-14_W7.62mm_Socket" H 5050 1150 50  0001 C CNN
 F 3 "" H 5050 1150 50  0001 C CNN
 F 4 "SN74HCT00N" H 5050 1150 60  0001 C CNN "MPN"
@@
 F 0 "U3" H 5050 1900 50  0000 C CNN
 F 1 "74HCT00" H 5050 1750 50  0000 C CNN
-F 2 "Housings_DIP:DIP-14_W7.62mm_Socket" H 5050 1850 50  0001 C CNN
+F 2 "rc2014:DIP-14_W7.62mm_Socket" H 5050 1850 50  0001 C CNN
 F 3 "" H 5050 1850 50  0001 C CNN
 	4    5050 1850
@@
 F 0 "C4" H 3625 6500 50  0000 L CNN
 F 1 "C" H 3625 6300 50  0000 L CNN
-F 2 "Capacitors_THT:C_Disc_D3.8mm_W2.6mm_P2.50mm" H 3638 6250 50  0001 C CNN
+F 2 "rc2014:C_Disc_D3.8mm_W2.6mm_P2.50mm" H 3638 6250 50  0001 C CNN
 F 3 "" H 3600 6400 50  0001 C CNN
 	1    3600 6400

Commit message: Rev 5 as sent to be manufactured
Parts:
- added JP7: USE !A4 FOR ENABLE, rc2014:Pin_Header_Straight_1x03_Pitch2.54mm, symbol Jumper_Dual
- C6, C7: footprint Capacitors_THT:CP_Radial_D6.3mm_P2.50mm -> rc2014:CP_Radial_D6.3mm_P2.50mm
Connections:
- wire segments 212 -> 217
Changed lines of the file:
@@
 Sheet 1 1
 Title "RC2014 YM2149 / AY-3-8910 sound card"
-Date "2017-05-13"
-Rev "3"
+Date "2017-07-16"
+Rev "5"
 Comp ""
 Comment1 ""
@@
 F 0 "C6" H 9025 900 50  0000 L CNN
 F 1 "470uF" H 9025 700 50  0000 L CNN
-F 2 "Capacitors_THT:CP_Radial_D6.3mm_P2.50mm" H 9038 650 50  0001 C CNN
+F 2 "rc2014:CP_Radial_D6.3mm_P2.50mm" H 9038 650 50  0001 C CNN
 F 3 "" H 9000 800 50  0000 C CNN
 	1    9000 800
@@
 F 0 "C7" H 9025 1100 50  0000 L CNN
 F 1 "470uF" H 9025 900 50  0000 L CNN
-F 2 "Capacitors_THT:CP_Radial_D6.3mm_P2.50mm" H 9038 850 50  0001 C CNN
+F 2 "rc2014:CP_Radial_D6.3mm_P2.50mm" H 9038 850 50  0001 C CNN
 F 3 "" H 9000 1000 50  0000 C CNN
 	1    9000 1000
@@
 Wire Wire Line
 	1950 1000 1700 1000
-Wire Wire Line
-	1950 1400 1700 1400
-Wire Wire Line
-	1950 1500 1700 1500
 Text Label 1750 1000 0    60   ~ 0
 A5
@@
 L Jumper_Dual JP1
 U 1 1 58DB01E6
-P 1100 1100
-F 0 "JP1" H 1100 1250 50  0000 C CNN
-F 1 "USE A4 FOR ENABLE" H 1150 800 50  0000 C CNN
-F 2 "rc2014:Pin_Header_Straight_1x03_Pitch2.54mm" H 1100 -100 50  0001 C CNN
-F 3 "" H 1100 -100 50  0001 C CNN
-F 4 "CONN 1x03" H 1100 1100 60  0001 C CNN "MPN"
-	1    1100 1100
-	1    0    0    -1
-$EndComp
-Wire Wire Line
-	1700 1400 1700 1600
+P 1100 950
+F 0 "JP1" H 950 1100 50  0000 C CNN
+F 1 "USE A4 FOR ENABLE" H 1100 1250 50  0000 C CNN
+F 2 "rc2014:Pin_Header_Straight_1x03_Pitch2.54mm" H 1100 -250 50  0001 C CNN
+F 3 "" H 1100 -250 50  0001 C CNN
+F 4 "CONN 1x03" H 1100 950 60  0001 C CNN "MPN"
+	1    1100 950
+	1    0    0    -1
+$EndComp
 $Comp
 L GND #PWR023
 U 1 1 58DB06C5
-P 1700 1600
-F 0 "#PWR023" H 1700 1350 50  0001 C CNN
-F 1 "GND" H 1700 1450 50  0000 C CNN
-F 2 "" H 1700 1600 50  0001 C CNN
-F 3 "" H 1700 1600 50  0001 C CNN
-	1    1700 1600
-	1    0    0    -1
-$EndComp
-Text Label 1400 1100 0    60   ~ 0
+P 850 1300
+F 0 "#PWR023" H 850 1050 50  0001 C CNN
+F 1 "GND" H 850 1150 50  0000 C CNN
+F 2 "" H 850 1300 50  0001 C CNN
+F 3 "" H 850 1300 50  0001 C CNN
+	1    850  1300
+	1    0    0    -1
+$EndComp
+Text Label 1400 1250 0    60   ~ 0
 A4
 $Comp
 L VCC #PWR024
 U 1 1 58DB09C6
-P 850 1100
-F 0 "#PWR024" H 850 950 50  0001 C CNN
-F 1 "VCC" H 850 1250 50  0000 C CNN
-F 2 "" H 850 1100 50  0001 C CNN
-F 3 "" H 850 1100 50  0001 C CNN
-	1    850  1100
+P 850 950
+F 0 "#PWR024" H 850 800 50  0001 C CNN
+F 1 "VCC" H 850 1100 50  0000 C CNN
+F 2 "" H 850 950 50  0001 C CNN
+F 3 "" H 850 950 50  0001 C CNN
+	1    850  950
 	0    -1   -1   0
 $EndComp
-Connection ~ 1700 1500
 Text Label 5750 1150 0    60   ~ 0
 CS
@@
 Wire Wire Line
 	2850 3550 2650 3550
-Wire Wire Line
-	1350 1100 1550 1100
-Wire Wire Line
-	1100 1300 1950 1300
-Wire Wire Line
-	1100 1300 1100 1200
 Wire Wire Line
 	2000 3200 1800 3200
@@
 Wire Bus Line
 	11000 1900 11000 3100
+$Comp
+L Jumper_Dual JP7
+U 1 1 596A80CC
+P 1100 1250
+F 0 "JP7" H 950 1400 50  0000 C CNN
+F 1 "USE !A4 FOR ENABLE" H 1100 950 50  0000 C CNN
+F 2 "rc2014:Pin_Header_Straight_1x03_Pitch2.54mm" H 1100 50  50  0001 C CNN
+F 3 "" H 1100 50  50  0001 C CNN
+F 4 "CONN 1x03" H 1100 1250 60  0001 C CNN "MPN"
+	1    1100 1250
+	1    0    0    -1
+$EndComp
+Wire Wire Line
+	1950 1500 1850 1500
+Wire Wire Line
+	1100 1100 1100 1050
+Wire Wire Line
+	1350 950  1500 950
+Text Label 1400 950  0    60   ~ 0
+A4
+Wire Wire Line
+	1550 1250 1350 1250
+Wire Wire Line
+	850  1250 850  1300
+Wire Wire Line
+	1950 1300 1700 1300
+Wire Wire Line
+	1700 1300 1700 1100
+Wire Wire Line
+	1700 1100 1100 1100
+Wire Wire Line
+	1850 1500 1850 1400
+Connection ~ 1850 1400
+Wire Wire Line
+	1950 1400 1100 1400
+Wire Wire Line
+	1100 1400 1100 1350
 $EndSCHEMATC

Commit message: WIP updating schematic
Parts:
- C1, C2, C3, C4, C5: symbol C -> Device:C
- C6, C7: symbol CP -> Device:C
- J1: symbol JACK_TRS_6PINS -> Connector:AudioJack3
- J2: symbol CONN_02X09 -> Connector_Generic:Conn_02x09_Odd_Even
- JP1, JP2, JP5, JP7: symbol Jumper_Dual -> Jumper:Jumper_3_Bridged12
- JP3: symbol CONN_02X03 -> Connector_Generic:Conn_02x03_Odd_Even
- JP4: symbol CONN_02X08 -> Connector_Generic:Conn_02x08_Odd_Even
- JP6: symbol Jumper -> Jumper:Jumper_2_Bridged
- P1: symbol CONN_01X39 -> Connector_Generic:Conn_01x39
- R1, R2, R3, R4, R5, R6: symbol R_Small -> Device:R_Small
- R7: footprint rc2014:R_Axial_DIN0207_L6.3mm_D2.5mm_P10.16mm_Horizontal -> (none); symbol R_Small -> Device:R_Small
- U1, U2: symbol 74LS138 -> 74xx:74LS138
- U3: symbol 74HCT00 -> 74xx:74HCT00
- U3: footprint rc2014:DIP-14_W7.62mm_Socket -> (none); symbol 74HCT00 -> 74xx:74HCT00; MPN SN74HCT00N -> (none); Supplier URL http://uk.farnell.com/texas-instruments/sn74hct00n/quad-2-i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 -> (none)
- U4: symbol 74LS74 -> 74xx:74LS74
- U5: symbol DIL40 -> rc2014-ym2149-rescue:DIL40
Connections:
- wire segments 217 -> 243
Other:
- moved on the sheet: U3A, U3B, U3C, U3D

Commit message: Work in progress converting to Kicad 5
Parts:
- added unit 5 of U3
- added unit 3 of U4
- J1: symbol Connector:AudioJack3 -> Connector:AudioJack3_Dual_Switch
- JP1, JP2, JP7: symbol Jumper:Jumper_3_Bridged12 -> jumper_dual:Jumper_Dual
- R7: footprint (none) -> rc2014:R_Axial_DIN0207_L6.3mm_D2.5mm_P10.16mm_Horizontal
- U3: footprint (none) -> rc2014:DIP-14_W7.62mm_Socket
- U4: Base number 74HCT74 -> (none); MPN SN74HCT74N -> (none); Supplier URL http://uk.farnell.com/texas-instruments/sn74hct74n/ic-flip-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 -> (none)
Connections:
- wire segments 243 -> 244
Changed lines of the file:
@@
 $EndComp
 $Comp
-L Connector:AudioJack3 J1
+L Connector:AudioJack3_Dual_Switch J1
 U 1 1 5898EEE9
-P 9950 900
-F 0 "J1" H 9950 1300 50  0000 C CNN
-F 1 "AUDIO OUT" H 9900 600 50  0000 C CNN
-F 2 "rc2014:cliff_fcr1295_socket" H 10050 750 50  0001 C CNN
-F 3 "" H 10050 750 50  0000 C CNN
-	1    9950 900
+P 10150 1100
+F 0 "J1" H 10150 1450 50  0000 C CNN
+F 1 "AUDIO OUT" H 10150 650 50  0000 C CNN
+F 2 "rc2014:cliff_fcr1295_socket" H 10250 950 50  0001 C CNN
+F 3 "" H 10250 950 50  0000 C CNN
+	1    10150 1100
 	-1   0    0    1
 $EndComp
@@
 L power:GND #PWR05
 U 1 1 5898F3AF
-P 9150 1300
-F 0 "#PWR05" H 9150 1050 50  0001 C CNN
-F 1 "GND" H 9150 1150 50  0000 C CNN
-F 2 "" H 9150 1300 50  0000 C CNN
-F 3 "" H 9150 1300 50  0000 C CNN
-	1    9150 1300
+P 9500 1500
+F 0 "#PWR05" H 9500 1250 50  0001 C CNN
+F 1 "GND" H 9500 1350 50  0000 C CNN
+F 2 "" H 9500 1500 50  0000 C CNN
+F 3 "" H 9500 1500 50  0000 C CNN
+	1    9500 1500
 	1    0    0    -1
 $EndComp
@@
 F 3 "" H 7800 3350 50  0000 C CNN
 	1    7800 3350
-	1    0    0    -1
-$EndComp
-$Comp
-L 74xx:74LS74 U4
-U 1 1 58ACAA95
-P 5700 5300
-F 0 "U4" H 5850 5600 50  0000 C CNN
-F 1 "74HCT74" H 6000 5005 50  0000 C CNN
-F 2 "rc2014:DIP-14_W7.62mm_Socket" H 5700 5300 50  0001 C CNN
-F 3 "" H 5700 5300 50  0000 C CNN
-F 4 "SN74HCT74N" H 5700 5300 60  0001 C CNN "MPN"
-F 5 "74HCT74" H 5700 5300 60  0001 C CNN "Base number"
-F 6 "http://uk.farnell.com/texas-instruments/sn74hct74n/ic-flip-flop-2-circuits/dp/1470823" H 5700 5300 60  0001 C CNN "Supplier URL"
-	1    5700 5300
 	1    0    0    -1
 $EndComp
@@
 F 1 "74HCT74" H 6000 6555 50  0000 C CNN
 F 2 "rc2014:DIP-14_W7.62mm_Socket" H 5700 6850 50  0001 C CNN
-F 3 "" H 5700 6850 50  0000 C CNN
+F 3 "74xx/74hc_hct74.pdf" H 5700 6850 50  0001 C CNN
 	2    5700 6850
 	1    0    0    -1
@@
 F 0 "R7" H 8330 1220 50  0000 L CNN
 F 1 "1K6" H 8330 1160 50  0000 L CNN
-F 2 "" H 8300 1200 50  0001 C CNN
+F 2 "rc2014:R_Axial_DIN0207_L6.3mm_D2.5mm_P10.16mm_Horizontal" H 8300 1200 50  0001 C CNN
 F 3 "~" H 8300 1200 50  0001 C CNN
 	1    8300 1200
@@
 	7350 4050 7350 4100
 Wire Wire Line
-	9150 1000 9600 1000
-Wire Wire Line
-	9150 800  9600 800
-Wire Wire Line
-	9150 1200 9150 1300
+	9500 1200 9500 1500
 Wire Wire Line
 	5950 2450 6250 2450
@@
 Wire Wire Line
 	1100 4900 1400 4900
-Wire Wire Line
-	9750 1100 9600 1100
-Wire Wire Line
-	9600 1100 9600 1000
-Connection ~ 9600 1000
-Wire Wire Line
-	9750 900  9600 900
-Wire Wire Line
-	9600 900  9600 800
-Connection ~ 9600 800
 Wire Wire Line
 	7450 5650 7450 5500
@@
 CS
 $Comp
-L Jumper:Jumper_3_Bridged12 JP2
+L jumper_dual:Jumper_Dual JP2
 U 1 1 58DB0BB0
 P 2250 3650
 F 0 "JP2" H 2250 3800 50  0000 C CNN
 F 1 "ENABLE SELECTOR" H 2250 3300 50  0000 C CNN
-F 2 "rc2014:Pin_Header_Straight_1x03_Pitch2.54mm" H 2250 2450 50  0001 C CNN
-F 3 "" H 2250 2450 50  0001 C CNN
+F 2 "rc2014:Pin_Header_Straight_1x03_Pitch2.54mm" H 2250 3650 50  0001 C CNN
+F 3 "~" H 2250 3650 50  0001 C CNN
 	1    2250 3650
 	1    0    0    -1
@@
 F 0 "U3" H 5050 1800 50  0000 C CNN
 F 1 "74HCT00" H 5050 1500 50  0000 C CNN
-F 2 "" H 5050 1750 50  0001 C CNN
+F 2 "rc2014:DIP-14_W7.62mm_Socket" H 5050 1750 50  0001 C CNN
 F 3 "http://www.ti.com/lit/gpn/sn74hct00" H 5050 1750 50  0001 C CNN
 	3    5050 1750
@@
 	3850 2150 3700 2150
 $Comp
-L Jumper:Jumper_3_Bridged12 JP7
+L jumper_dual:Jumper_Dual JP7
 U 1 1 596A80CC
 P 1100 1900
@@
 	7300 1600 7600 1600
 Wire Wire Line
-	9600 1000 9750 1000
-Wire Wire Line
-	9600 800  9750 800
-Wire Wire Line
 	2700 3200 2700 3300
 Wire Wire Line
@@
 Wire Wire Line
 	3850 1850 4350 1850
-Wire Wire Line
-	9750 1300 9600 1300
-Wire Wire Line
-	9600 1200 9750 1200
-Wire Wire Line
-	9150 1200 9600 1200
-Connection ~ 9600 1200
-Wire Wire Line
-	9600 1300 9600 1200
 $Comp
 L power:GND #PWR0101
@@
 Wire Wire Line
 	850  1550 750  1550
-Wire Wire Line
-	2250 3800 2250 3850
-Wire Wire Line
-	2250 3850 2950 3850
 Wire Wire Line
 	1100 5100 4250 5100
@@
 $EndComp
 $Comp
-L Jumper:Jumper_3_Bridged12 JP1
+L jumper_dual:Jumper_Dual JP1
 U 1 1 58DB01E6
 P 1100 1550
@@
 	-1   0    0    1
 $EndComp
+Wire Wire Line
+	2250 3850 2950 3850
+Wire Wire Line
+	2250 3750 2250 3850
+Wire Wire Line
+	1100 2000 1100 2050
+Wire Wire Line
+	9150 800  9600 800
+Wire Wire Line
+	9500 1200 9600 1200
+Wire Wire Line
+	9150 1000 9600 1000
+Wire Wire Line
+	9600 800  9600 900
+Wire Wire Line
+	9600 900  9950 900
+Connection ~ 9600 800
+Wire Wire Line
+	9600 800  9950 800
+Wire Wire Line
+	9600 1000 9600 1100
+Wire Wire Line
+	9600 1100 9950 1100
+Connection ~ 9600 1000
+Wire Wire Line
+	9600 1000 9950 1000
+Wire Wire Line
+	9600 1200 9600 1300
+Wire Wire Line
+	9600 1300 9950 1300
+Connection ~ 9600 1200
+Wire Wire Line
+	9600 1200 9950 1200
+$Comp
+L 74xx:74LS74 U4
+U 1 1 58ACAA95
+P 5700 5300
+F 0 "U4" H 5850 5600 50  0000 C CNN
+F 1 "74HCT74" H 6000 5005 50  0000 C CNN
+F 2 "rc2014:DIP-14_W7.62mm_Socket" H 5700 5300 50  0001 C CNN
+F 3 "74xx/74hc_hct74.pdf" H 5700 5300 50  0001 C CNN
+	1    5700 5300
+	1    0    0    -1
+$EndComp
+$Comp
+L 74xx:74HC74 U4
+U 3 1 5EA440B3
+P 4250 6500
+F 0 "U4" H 4480 6546 50  0000 L CNN
+F 1 "74HCT74" H 4480 6455 50  0000 L CNN
+F 2 "rc2014:DIP-14_W7.62mm_Socket" H 4250 6500 50  0001 C CNN
+F 3 "74xx/74hc_hct74.pdf" H 4250 6500 50  0001 C CNN
+	3    4250 6500
+	1    0    0    -1
+$EndComp
+$Comp
+L power:VCC #PWR028
+U 1 1 5EA44D62
+P 4250 6100
+F 0 "#PWR028" H 4250 5950 50  0001 C CNN
+F 1 "VCC" H 4250 6250 50  0000 C CNN
+F 2 "" H 4250 6100 50  0000 C CNN
+F 3 "" H 4250 6100 50  0000 C CNN
+	1    4250 6100
+	1    0    0    -1
+$EndComp
+$Comp
+L power:GND #PWR029
+U 1 1 5EA45373
+P 4250 6900
+F 0 "#PWR029" H 4250 6650 50  0001 C CNN
+F 1 "GND" H 4250 6750 50  0000 C CNN
+F 2 "" H 4250 6900 50  0001 C CNN
+F 3 "" H 4250 6900 50  0001 C CNN
+	1    4250 6900
+	1    0    0    -1
+$EndComp
 Wire Bus Line
 	6000 4200 9950 4200
@@
 Wire Bus Line
 	6000 2750 6000 4200
+$Comp
+L 74xx:74HCT00 U3
+U 5 1 5EA6DD08
+P 4800 1050
+F 0 "U3" V 4433 1050 50  0000 C CNN
+F 1 "74HCT00" V 4524 1050 50  0000 C CNN
+F 2 "" H 4800 1050 50  0001 C CNN
+F 3 "http://www.ti.com/lit/gpn/sn74hct00" H 4800 1050 50  0001 C CNN
+	5    4800 1050
+	0    1    1    0
+$EndComp
+$Comp
+L power:GND #PWR?
+U 1 1 5EA780C6
+P 4300 1050
+F 0 "#PWR?" H 4300 800 50  0001 C CNN
+F 1 "GND" H 4300 900 50  0000 C CNN
+F 2 "" H 4300 1050 50  0001 C CNN
+F 3 "" H 4300 1050 50  0001 C CNN
+	1    4300 1050
+	1    0    0    -1
+$EndComp
+$Comp
+L power:VCC #PWR?
+U 1 1 5EA78A23
+P 5300 1050
+F 0 "#PWR?" H 5300 900 50  0001 C CNN
+F 1 "VCC" H 5300 1200 50  0000 C CNN
+F 2 "" H 5300 1050 50  0000 C CNN
+F 3 "" H 5300 1050 50  0000 C CNN
+	1    5300 1050
+	1    0    0    -1
+$EndComp
 $EndSCHEMATC

Commit message: Update for Kicad 5 complete
Parts:
- removed U5: AY-3-8190/YM2149F, rc2014:DIP-40_W15.24mm_Socket, symbol rc2014-ym2149-rescue:DIL40
- added U5: YM2149, rc2014:DIP-40_W15.24mm_Socket, symbol Audio:YM2149
- JP5: symbol Jumper:Jumper_3_Bridged12 -> jumper_dual:Jumper_Dual
- U3: footprint (none) -> rc2014:DIP-14_W7.62mm_Socket
Connections:
- wire segments 244 -> 236
- no-connect marks 24 -> 22
Other:
- moved on the sheet: C1, C2, C3, C4, C5, J2, JP6, U4A, U4B, U4C
