File: rc2014-ym2149.sch (KiCad schematic (older format))
At the start: 29 parts, among them J1 AUDIO OUT, J2 IO Out, P1 RC2014 BUS, U1 74HCT138, U2 74HCT138, U3 74HCT00, U4 74HCT74, U5 YM2149

Commit message: Initial rev 6
Parts:
- removed J1: AUDIO OUT, rc2014:cliff_fcr1295_socket, symbol Connector:AudioJack3_Dual_Switch
- removed JP3: CONN_02X03, rc2014:Pin_Header_Straight_2x03_Pitch2.54mm, symbol Connector_Generic:Conn_02x03_Odd_Even
- added CON1: SJ1-3523N, rc2014:Headphone_Jack_3.5mm_5_pin, symbol Connector:AudioJack3_SwitchTR
- added JP3: MSX/ZX Spectrum, Connector_PinHeader_2.54mm:PinHeader_1x03_P2.54mm_Vertical, symbol jumper_dual:Jumper_Dual
- added JP8: Bus clock, Connector_PinHeader_2.54mm:PinHeader_1x03_P2.54mm_Vertical, symbol jumper_dual:Jumper_Dual
- added X1: CXO_DIP8, Oscillator:Oscillator_DIP-8, symbol Oscillator:CXO_DIP8
- C1, C2, C3, C4, C5: footprint rc2014:C_Disc_D3.8mm_W2.6mm_P2.50mm -> Capacitor_THT:C_Disc_D3.8mm_W2.6mm_P2.50mm
- C6, C7: footprint rc2014:CP_Radial_D6.3mm_P2.50mm -> Capacitor_THT:CP_Radial_D6.3mm_P2.50mm
- J2: footprint rc2014:Pin_Header_Straight_2x09_Pitch2.54mm -> Connector_PinHeader_2.54mm:PinHeader_2x09_P2.54mm_Vertical
- JP1: value USE A4 FOR ENABLE -> MSX/ZX Spectrum; footprint rc2014:Pin_Header_Straight_1x03_Pitch2.54mm -> Connector_PinHeader_2.54mm:PinHeader_1x03_P2.54mm_Vertical
- JP2: value ENABLE SELECTOR -> MSX/ZX Spectrum; footprint rc2014:Pin_Header_Straight_1x03_Pitch2.54mm -> Connector_PinHeader_2.54mm:PinHeader_1x03_P2.54mm_Vertical; MPN (none) -> CONN 1x03
- JP4: footprint rc2014:Pin_Header_Straight_2x08_Pitch2.54mm -> Connector_PinHeader_2.54mm:PinHeader_2x09_P2.54mm_Vertical; symbol Connector_Generic:Conn_02x08_Odd_Even -> Connector_Generic:Conn_02x09_Odd_Even
- JP5: footprint rc2014:Pin_Header_Straight_1x03_Pitch2.54mm -> Connector_PinHeader_2.54mm:PinHeader_1x03_P2.54mm_Vertical
- JP6: footprint rc2014:Pin_Header_Straight_1x02_Pitch2.54mm -> Connector_PinHeader_2.54mm:PinHeader_1x02_P2.54mm_Vertical
- JP7: value USE !A4 FOR ENABLE -> Upper/lower half; footprint rc2014:Pin_Header_Straight_1x03_Pitch2.54mm -> Connector_PinHeader_2.54mm:PinHeader_1x03_P2.54mm_Vertical
- P1: footprint rc2014:Pin_Header_Straight_1x39_Pitch2.54mm_NoSilk -> Connector_PinHeader_2.54mm:PinHeader_1x39_P2.54mm_Vertical
- R1, R2, R3, R4, R5, R6, R7: footprint rc2014:R_Axial_DIN0207_L6.3mm_D2.5mm_P10.16mm_Horizontal -> Resistor_THT:R_Axial_DIN0207_L6.3mm_D2.5mm_P10.16mm_Horizontal
- U1, U2: footprint rc2014:DIP-16_W7.62mm_Socket -> Package_DIP:DIP-16_W7.62mm_Socket_LongPads
- U3, U4: footprint rc2014:DIP-14_W7.62mm_Socket -> Package_DIP:DIP-14_W7.62mm_Socket_LongPads
- U5: footprint rc2014:DIP-40_W15.24mm_Socket -> Package_DIP:DIP-40_W15.24mm_Socket_LongPads
Connections:
- net labels added: ~CS, ~IORQ, ~RD, ~RESET, ~WR
- net labels removed: /IORQ, /RD, /RESET, /SEL, /WR, /YM_A9, BC2, CLOCK, CS, REG, YM_A8
- wire segments 236 -> 228
- no-connect marks 22 -> 20
Other:
- moved on the sheet: JP7, U1, U3A, U3C, U3D, U3E
